File: pcb/ads1115/screen_sensors_draft.kicad_pcb (KiCad board)
At the start: 2 copper layers, 42 x 32 mm, 16 parts, among them J1 WAVESHARE_I2C, J2 BOILER_PROBE, J3 XDB401_ANALOG, U1 ADS1115IDGSR, U2 SHT40-AD1B

Commit message: pcb manual rework
Parts:
- moved C6 10.5 mm to (124.1, 118.5), turned to -90 degrees
- moved H2 9.87 mm to (129.1, 106.5)
- moved R3 9.62 mm to (118.5, 121.5)
- moved U2 9.59 mm to (127.5, 116.3), turned to -90 degrees
- moved H4 9.40 mm to (129.1, 128.5)
- moved C4 8.06 mm to (120.0, 121.5), turned to -90 degrees
- moved C1 5.39 mm to (122.0, 118.5), turned to -90 degrees
- moved C2 4.55 mm to (109.1, 114.5), turned to 90 degrees
- moved J1 3.72 mm to (114.1, 107.0)
- moved U1 3.72 mm to (117.6, 117.5)
- moved J3 3.40 mm to (114.1, 127.0)
- moved H1 3.00 mm to (103.6, 106.5)
- moved C5 2.79 mm to (114.6, 123.0), turned to 0 degrees
- moved R1 2.45 mm to (109.1, 117.5), turned to -90 degrees
- moved J2 1.08 mm to (105.1, 115.0), turned to -90 degrees
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Connections:
- J1 pad 3: /SDA -> /SCL
- J1 pad 4: /SCL -> /SDA
Routing:
- net /GND: track 95.3 -> 28.5 mm, vias 8 -> 6
- net /3V3: track 85.8 -> 49.3 mm, vias 3 -> 4
- net /BOILER_ADC: track 18.2 -> 11.4 mm, vias 2 -> 0
- net /PRESS_ADC: track 9.83 -> 3.85 mm, vias 2 -> 0
- net /PRESS_SIGNAL: track 8.73 -> 4.92 mm, vias 1 -> 0
- net /SCL: track 23.6 -> 20.2 mm, vias 2 -> 0
- net /SDA: track 26.1 -> 23.4 mm, vias 1 -> 2
Other:
- board size 42 x 32 mm -> 32.5 x 29 mm
- board text removed: "CoffeeFlow"

Commit message: Screen Sensors PCB
Parts:
- moved C2 3.98 mm to (111.0, 111.0), turned to 180 degrees
- moved C5 3.44 mm to (127.5, 118.0), turned to 0 degrees
- moved H2 2.79 mm to (126.5, 105.5)
- moved H4 2.60 mm to (126.5, 128.5)
- moved J1 2.49 mm to (111.8, 106.0)
- moved C3 1.12 mm to (119.5, 120.5)
- moved R3 1.12 mm to (118.0, 120.5)
- moved C4 1.08 mm to (115.0, 122.0)
- moved R1 1.08 mm to (109.5, 116.5), turned to 0 degrees
- moved U2 1.00 mm to (127.6, 115.3)
- moved J3 1.00 mm to (113.1, 127.0)
- moved H1 1.00 mm to (103.6, 105.5)
- moved U1 1.00 mm to (117.6, 116.5)
- renumbered C4 to C3, C5 to C4, C6 to C5
Routing:
- net /GND: track 28.5 -> 20.1 mm, vias 6 -> 8
- net /3V3: track 49.3 -> 56.1 mm
- net /PRESS_SIGNAL: track 4.92 -> 5.83 mm
- net /SDA: track 23.4 -> 24.1 mm
Other:
- board size 32.5 x 29 mm -> 30 x 30 mm
- board text added: "RH/T"
- board text removed: "RH / T"

Commit message: pcb update
Parts:
- added POWER: RED / POWER, LED_SMD:LED_0603_1608Metric, F.Cu at (106.0, 111.0)
- added R4: 2.2k, Resistor_SMD:R_0603_1608Metric, F.Cu at (109.5, 111.0)
- moved C2 2.50 mm to (113.5, 111.0), turned to 0 degrees
Routing:
- net /GND: track 20.1 -> 23.7 mm
- net /3V3: track 56.1 -> 58.3 mm
- net Net-(D1-A): track 0.00 -> 1.89 mm
Other:
- board text added: "4.7K"

Commit message: Use basic pressure resistor and add JLCPCB manufacturing exporter
Parts:
- R3: value 1k 0.1% -> 1k
Changed lines of the file:
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@@
 			)
 		)
-		(property "Value" "1k 0.1%"
+		(property "Value" "1k"
 			(at 0 1.43 90)
 			(layer "F.Fab")
@@
 			)
 		)
-		(property "MPN" "PTFR0603B1K00N9"
+		(property "MPN" "0603WAF1001T5E"
 			(at 0 0 0)
 			(layer "F.SilkS")
@@
 			)
 		)
-		(property "LCSC" "C394536"
+		(property "LCSC" "C21190"
 			(at 0 0 0)
 			(layer "F.SilkS")
