File: pcb/screen_sensors/screen_sensors.kicad_pcb (KiCad board)
At the start: 2 copper layers, 30 x 30 mm, 18 parts, among them J1 WAVESHARE_I2C, J2 BOILER_PROBE, J3 XDB401_ANALOG, U1 ADS1115IDGSR, U2 SHT40-AD1B

Commit message: pcb sensors: ground plane
Routing:
- net /GND: track 23.7 -> 14.9 mm, vias 8 -> 7
- added copper zone on F.Cu, net /GND
Changed lines of the file:
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@@
+	)
+	(segment
+		(start 122 119.275)
+		(end 122 120.5)
+		(width 0.2)
+		(layer "F.Cu")
+		(net "/GND")
+	)
+	(segment
+		(start 110.325 116.5)
+		(end 111.5 116.5)
+		(width 0.2)
+		(layer "F.Cu")
+		(net "/GND")
+	)
+	(segment
+		(start 115.599911 126.975)
+		(end 115.599911 126.400089)
+		(width 0.2)
+		(layer "F.Cu")
+		(net "/GND")
+	)
+	(segment
+		(start 114.324911 106)
+		(end 114.324911 106.675089)
+		(width 0.2)
+		(layer "F.Cu")
+		(net "/GND")
+	)
+	(segment
+		(start 115.449911 115.5)
+		(end 114.5 115.5)
+		(width 0.2)
+		(layer "F.Cu")
+		(net "/GND")
+	)
+	(segment
+		(start 115.775 121.275)
+		(end 115.5 121)
+		(width 0.2)
+		(layer "F.Cu")
+		(net "/GND")
+	)
+	(segment
+		(start 114.5 116.5)
+		(end 114 116)
+		(width 0.2)
+		(layer "F.Cu")
+		(net "/GND")
+	)
+	(segment
+		(start 128 117.725)
+		(end 128.275 118)
+		(width 0.2)
+		(layer "F.Cu")
+		(net "/GND")
+	)
+	(segment
+		(start 128 116)
+		(end 128 117.725)
+		(width 0.2)
+		(layer "F.Cu")
+		(net "/GND")
+	)
+	(segment
+		(start 115.449911 116.5)
+		(end 114.5 116.5)
+		(width 0.2)
+		(layer "F.Cu")
+		(net "/GND")
+	)
+	(segment
+		(start 114.5 115.5)
+		(end 114 116)
+		(width 0.2)
+		(layer "F.Cu")
+		(net "/GND")
+	)
+	(segment
+		(start 105.2125 111)
+		(end 104 111)
+		(width 0.2)
+		(layer "F.Cu")
+		(net "/GND")
+	)
+	(segment
+		(start 115.775 122)
+		(end 115.775 121.275)
+		(width 0.2)
+		(layer "F.Cu")
+		(net "/GND")
+	)
+	(segment
+		(start 114.275 111)
+		(end 115.5 111)
+		(width 0.2)
+		(layer "F.Cu")
+		(net "/GND")
+	)
+	(segment
+		(start 128.275 118)
+		(end 128.275 120.275)
+		(width 0.2)
+		(layer "F.Cu")
+		(net "/GND")
+	)
+	(via
+		(at 114 116)
+		(size 0.6)
+		(drill 0.3)
+		(layers "F.Cu" "B.Cu")
+		(free yes)
+		(net "/GND")
+	)
+	(via
+		(at 104 111)
+		(size 0.6)
+		(drill 0.3)
+		(layers "F.Cu" "B.Cu")
+		(free yes)
+		(net "/GND")
+	)
+	(via
+		(at 111.5 116.5)
+		(size 0.6)
+		(drill 0.3)
+		(layers "F.Cu" "B.Cu")
+		(free yes)
+		(net "/GND")
+	)
+	(via
+		(at 128.275 120.275)
+		(size 0.6)
+		(drill 0.3)
+		(layers "F.Cu" "B.Cu")
+		(net "/GND")
+	)
+	(via
+		(at 122 120.5)
+		(size 0.6)
+		(drill 0.3)
+		(layers "F.Cu" "B.Cu")
+		(free yes)
+		(net "/GND")
+	)
+	(via
+		(at 115.5 111)
+		(size 0.6)
+		(drill 0.3)
+		(layers "F.Cu" "B.Cu")
+		(free yes)
+		(net "/GND")
+	)
+	(via
+		(at 115.5 121)
+		(size 0.6)
+		(drill 0.3)
+		(layers "F.Cu" "B.Cu")
+		(free yes)
+		(net "/GND")
+	)
+	(segment
+		(start 108.675 111)
+		(end 106.7875 111)
+		(width 0.2)
+		(layer "F.Cu")
+		(net "Net-(POWER-A)")
 	)
 	(segment
@@
 	)
 	(segment
-		(start 115.775 123.225)
-		(end 115.5 123.5)
-		(width 0.2)
-		(layer "F.Cu")
-		(net "/GND")
-	)
-	(segment
-		(start 114.275 108.049911)
-		(end 114.324911 108)
-		(width 0.2)
-		(layer "F.Cu")
-		(net "/GND")
-	)
-	(segment
-		(start 115.599911 123.599911)
-		(end 115.5 123.5)
-		(width 0.2)
-		(layer "F.Cu")
-		(net "/GND")
-	)
-	(segment
-		(start 114.324911 106)
-		(end 114.324911 108)
-		(width 0.2)
-		(layer "F.Cu")
-		(net "/GND")
-	)
-	(segment
-		(start 114.275 111)
-		(end 114.275 108.049911)
-		(width 0.2)
-		(layer "F.Cu")
-		(net "/GND")
-	)
-	(segment
-		(start 110.325 116.5)
-		(end 111 116.5)
-		(width 0.2)
-		(layer "F.Cu")
-		(net "/GND")
-	)
-	(segment
-		(start 115.775 122)
-		(end 115.775 123.225)
-		(width 0.2)
-		(layer "F.Cu")
-		(net "/GND")
-	)
-	(segment
-		(start 115.449911 115.5)
-		(end 114.5 115.5)
-		(width 0.2)
-		(layer "F.Cu")
-		(net "/GND")
-	)
-	(segment
-		(start 111 116.5)
-		(end 111.5 116)
-		(width 0.2)
-		(layer "F.Cu")
-		(net "/GND")
-	)
-	(segment
-		(start 114.5 116.5)
-		(end 114 116)
-		(width 0.2)
-		(layer "F.Cu")
-		(net "/GND")
-	)
-	(segment
-		(start 122 119.275)
-		(end 122 120.5)
-		(width 0.2)
-		(layer "F.Cu")
-		(net "/GND")
-	)
-	(segment
-		(start 128.275 118)
-		(end 128.275 120.275)
-		(width 0.2)
-		(layer "F.Cu")
-		(net "/GND")
-	)
-	(segment
-		(start 119.5 121.275)
-		(end 119.5 122.5)
-		(width 0.2)
-		(layer "F.Cu")
-		(net "/GND")
-	)
-	(segment
-		(start 105.2125 111)
-		(end 103.5 111)
-		(width 0.2)
-		(layer "F.Cu")
-		(net "/GND")
-	)
-	(segment
-		(start 128 117.725)
-		(end 128.275 118)
-		(width 0.2)
-		(layer "F.Cu")
-		(net "/GND")
-	)
-	(segment
-		(start 128 116)
-		(end 128 117.725)
-		(width 0.2)
-		(layer "F.Cu")
-		(net "/GND")
-	)
-	(segment
-		(start 115.449911 116.5)
-		(end 114.5 116.5)
-		(width 0.2)
-		(layer "F.Cu")
-		(net "/GND")
-	)
-	(segment
-		(start 114.5 115.5)
-		(end 114 116)
-		(width 0.2)
-		(layer "F.Cu")
-		(net "/GND")
-	)
-	(segment
-		(start 115.599911 126.975)
-		(end 115.599911 123.599911)
-		(width 0.2)
-		(layer "F.Cu")
-		(net "/GND")
-	)
-	(segment
-		(start 128.275 120.275)
-		(end 128.5 120.5)
-		(width 0.2)
-		(layer "F.Cu")
-		(net "/GND")
-	)
-	(via
-		(at 115.5 123.5)
-		(size 0.6)
-		(drill 0.3)
-		(layers "F.Cu" "B.Cu")
-		(free yes)
-		(net "/GND")
-	)
-	(via
-		(at 103.5 111)
-		(size 0.6)
-		(drill 0.3)
-		(layers "F.Cu" "B.Cu")
-		(free yes)
-		(net "/GND")
-	)
-	(via
-		(at 114 116)
-		(size 0.6)
-		(drill 0.3)
-		(layers "F.Cu" "B.Cu")
-		(free yes)
-		(net "/GND")
-	)
-	(via
-		(at 122 120.5)
-		(size 0.6)
-		(drill 0.3)
-		(layers "F.Cu" "B.Cu")
-		(net "/GND")
-	)
-	(via
-		(at 111.5 116)
-		(size 0.6)
-		(drill 0.3)
-		(layers "F.Cu" "B.Cu")
-		(free yes)
-		(net "/GND")
-	)
-	(via
-		(at 114.324911 108)
-		(size 0.6)
-		(drill 0.3)
-		(layers "F.Cu" "B.Cu")
-		(free yes)
-		(net "/GND")
-	)
-	(via
-		(at 128.5 120.5)
-		(size 0.6)
-		(drill 0.3)
-		(layers "F.Cu" "B.Cu")
-		(free yes)
-		(net "/GND")
-	)
-	(via
-		(at 119.5 122.5)
-		(size 0.6)
-		(drill 0.3)
-		(layers "F.Cu" "B.Cu")
-		(free yes)
-		(net "/GND")
-	)
-	(segment
 		(start 126.732843 114.032843)
 		(end 127.2 114.5)
@@
 		(net "/BOILER_ADC")
 	)
-	(segment
-		(start 108.675 111)
-		(end 106.7875 111)
-		(width 0.2)
-		(layer "F.Cu")
-		(net "Net-(POWER-A)")
-	)
 	(zone
+		(net "/GND")
+		(layer "F.Cu")
+		(name "GND top")
+		(hatch edge 0.5)
+		(connect_pads
+			(clearance 0.2)
+		)
+		(min_thickness 0.25)
+		(fill yes
+			(thermal_gap 0.25)
+			(thermal_bridge_width 0.25)
+			(island_removal_mode 0)
+		)
+		(polygon
+			(pts
+				(xy 100.599911 102.5) (xy 129.5 102.5) (xy 129.5 111.5) (xy 123.099911 111.5) (xy 123.099911 119.5)
+				(xy 129.5 119.5) (xy 129.5 131.5) (xy 100.599911 131.5)
+			)
+		)
+	)
+	(zone
