File: pcb/sensors/sensors.kicad_sch (KiCad schematic)
At the start: 22 parts, among them J1 POWER / 5V RECOM, J2 USB-C FLASH, SW1 BOOT, SW2 RESET, U1 ESP32-S3-MINI-1U-N8, U2 AMS1117-3.3

Commit message: pcb sensors: update
Parts:
- removed R1: 270, Resistor_SMD:R_0603_1608Metric, symbol Device:R
Other:
- note added: "C3: solid tantalum for AMS1117 stability. Provide copper heatsinking: 0.85W at 500mA; verify enclosure temperature. USB VBUS and J1 feed +5V: NEVER connect both power sources."
- note removed: "C3: solid tantalum for AMS1117 stability. R1: 12mA minimum-load bleeder. Provide copper heatsinking: 0.85W at 500mA; verify enclosure temperature. USB VBUS and J1 feed +5V: NEVER connect both power sources."
Changed lines of the file:
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@@
 (global_label "GND" (shape bidirectional) (at 144.78 91.44 0) (effects (font (size 1.0 1.0)) (justify left)) (property "Intersheetrefs" "${INTERSHEET_REFS}" (at 144.78 91.44 0) (hide yes) (effects (font (size 1.0 1.0)))))
 (symbol (lib_id "Device:C_Polarized") (at 144.78 82.55 0) (unit 1) (exclude_from_sim no) (in_bom yes) (on_board yes) (dnp no) (property "Reference" "C3" (at 149.78 80.55 0) (effects (font (size 1.1 1.1)) (justify left))) (property "Value" "22uF tantalum / 10V" (at 149.78 83.55 0) (effects (font (size 1.0 1.0)) (justify left))) (property "Footprint" "Capacitor_Tantalum_SMD:CP_EIA-3528-21_Kemet-B" (at 144.78 82.55 0) (effects (font (size 1.0 1.0)) (justify left)) (hide yes)) (property "Datasheet" "" (at 144.78 82.55 0) (effects (font (size 1.0 1.0)) (justify left)) (hide yes)) (property "Description" "Polarized capacitor" (at 144.78 82.55 0) (effects (font (size 1.0 1.0)) (justify left)) (hide yes)) (property "MPN" "22uF 10V solid tantalum, case B" (at 144.78 82.55 0) (effects (font (size 1.0 1.0)) (justify left)) (hide yes)) (pin "1") (pin "2") (instances (project "sensors" (path "/655ba0f3-0427-5cf4-88d9-0bb38b1023d4" (reference "C3") (unit 1)))))
-(wire (pts (xy 190.5 78.74) (xy 190.5 73.66)) (stroke (width 0) (type default)))
-(global_label "+3V3" (shape bidirectional) (at 190.5 73.66 0) (effects (font (size 1.0 1.0)) (justify left)) (property "Intersheetrefs" "${INTERSHEET_REFS}" (at 190.5 73.66 0) (hide yes) (effects (font (size 1.0 1.0)))))
-(wire (pts (xy 190.5 86.36) (xy 190.5 91.44)) (stroke (width 0) (type default)))
-(global_label "GND" (shape bidirectional) (at 190.5 91.44 0) (effects (font (size 1.0 1.0)) (justify left)) (property "Intersheetrefs" "${INTERSHEET_REFS}" (at 190.5 91.44 0) (hide yes) (effects (font (size 1.0 1.0)))))
-(symbol (lib_id "Device:R") (at 190.5 82.55 0) (unit 1) (exclude_from_sim no) (in_bom yes) (on_board yes) (dnp no) (property "Reference" "R1" (at 195.5 80.55 0) (effects (font (size 1.1 1.1)) (justify left))) (property "Value" "270" (at 195.5 83.55 0) (effects (font (size 1.0 1.0)) (justify left))) (property "Footprint" "Resistor_SMD:R_0603_1608Metric" (at 190.5 82.55 0) (effects (font (size 1.0 1.0)) (justify left)) (hide yes)) (property "Datasheet" "" (at 190.5 82.55 0) (effects (font (size 1.0 1.0)) (justify left)) (hide yes)) (property "Description" "Resistor" (at 190.5 82.55 0) (effects (font (size 1.0 1.0)) (justify left)) (hide yes)) (property "MPN" "Generic 270 1% 0603" (at 190.5 82.55 0) (effects (font (size 1.0 1.0)) (justify left)) (hide yes)) (pin "1") (pin "2") (instances (project "sensors" (path "/655ba0f3-0427-5cf4-88d9-0bb38b1023d4" (reference "R1") (unit 1)))))
-(text "C3: solid tantalum for AMS1117 stability. R1: 12mA minimum-load bleeder.\nProvide copper heatsinking: 0.85W at 500mA; verify enclosure temperature.\nUSB VBUS and J1 feed +5V: NEVER connect both power sources." (at 18 106 0) (effects (font (size 1.25 1.25)) (justify left top)))
+(text "C3: solid tantalum for AMS1117 stability.\nProvide copper heatsinking: 0.85W at 500mA; verify enclosure temperature.\nUSB VBUS and J1 feed +5V: NEVER connect both power sources." (at 18 106 0) (effects (font (size 1.25 1.25)) (justify left top)))
 (wire (pts (xy 35.56 124.46) (xy 35.56 129.54)) (stroke (width 0) (type default)))
 (global_label "+5V" (shape bidirectional) (at 35.56 129.54 0) (effects (font (size 1.0 1.0)) (justify left)) (property "Intersheetrefs" "${INTERSHEET_REFS}" (at 35.56 129.54 0) (hide yes) (effects (font (size 1.0 1.0)))))

Commit message: manual PCB design
Parts:
- J1: value POWER / 5V RECOM -> 5V POWER
- J2: footprint Connector_USB:USB_C_Receptacle_GCT_USB4105-xx-A_16P_TopMnt_Horizontal -> Sensors_Local:USB_C_Receptacle_GCT_USB4105-xx-A_16P_TopMnt_Horizontal_RoundedGND
- SW1, SW2: footprint Button_Switch_SMD:SW_SPST_TL3342 -> Button_Switch_SMD:SW_SPST_TS-1088-xR020
Connections:
- net CAN_RX: now also U1.14 (IO10); no longer U1.12 (IO8)
- net CAN_TX: now also U1.15 (IO11); no longer U1.11 (IO7)
- net FLOW_PULSE: now also U1.37 (IO41); no longer U1.8 (IO4)
- net HEATER_CMD: now also U1.16 (IO12); no longer U1.14 (IO10)
- net USB_HOST_DM: now also D1.1; no longer D1.2
- net USB_HOST_DP: now also D1.2; no longer D1.1
- net VALVE_CMD: now also U1.32 (IO36); no longer U1.13 (IO9)

Commit message: Finalize sensors PCB and JLCPCB manufacturing exports
Parts:
- added D2: GREEN / STATUS, LED_SMD:LED_0603_1608Metric, symbol Device:LED
- added R25: 1k, Resistor_SMD:R_0603_1608Metric, symbol Device:R
- C1: LCSC (none) -> C107365; MPN Generic 4.7uF X7R >=10V -> CL21B475KOFNNNE
- C2, C5: LCSC (none) -> C14663; MPN Generic 100nF X7R >=10V -> CC0603KRX7R9BB104
- C3: LCSC (none) -> C7198; MPN 22uF 10V solid tantalum, case B -> TAJB226K010RNJ
- C4: LCSC (none) -> C95841; MPN Generic 10uF X7R >=10V -> CL21B106KOQNNNE
- C6: LCSC (none) -> C29936; MPN Generic 1uF X7R >=10V -> CL10B105KA8NNNC
- D1: LCSC (none) -> C1855726
- J1: LCSC (none) -> C158012; MPN JST B2B-XH-A -> B2B-XH-A(LF)(SN)
- J2: LCSC (none) -> C3025063; MPN GCT USB4105-GF-A -> USB4105-GF-A-060
- R2, R23, R24, R3: LCSC (none) -> C25804; MPN Generic 10k 1% 0603 -> 0603WAF1002T5E
- R4, R5: LCSC (none) -> C23186; MPN Generic 5.1k 1% 0603 -> 0603WAF5101T5E
- R6, R7: LCSC (none) -> C23345; MPN Generic 22 1% 0603 -> 0603WAF220JT5E
- SW1, SW2: LCSC (none) -> C720477; MPN E-Switch TL3342F160QG -> TS-1088-AR02016
- U1: LCSC (none) -> C2980299
- U2: LCSC (none) -> C6186
Connections:
- net GND: now also D2.1 (K)
- net STATUS_LED: now reaches U1.34 (IO38)
- net STATUS_LED: now also R25.1
- new net STATUS_LED_A: D2.2 (A), R25.2
- no-connect marks 29 -> 28
Other:
- note added: "GPIO38 / pad34 HIGH = LED on"
Changed lines of the file:
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@@
 		(at 325.12 64.77)
 	)
-	(no_connect
-		(at 325.12 77.47)
-	)
 	(wire
 		(pts
@@
 			)
 		)
+		(property "LCSC" "C2980299" (at 309.88 72.39 0) (hide yes) (effects (font (size 1 1))))
 	)
 	(symbol
@@
 			)
 		)
-		(property "MPN" "Generic 1uF X7R >=10V"
+		(property "MPN" "CL10B105KA8NNNC"
 			(at 384.81 124.46 0)
 			(hide yes)
@@
 			)
 		)
+		(property "LCSC" "C29936" (at 384.81 124.46 0) (hide yes) (effects (font (size 1 1))))
 	)
 	(symbol
@@
 			)
 		)
-		(property "MPN" "JST B2B-XH-A"
+		(property "MPN" "B2B-XH-A(LF)(SN)"
 			(at 39.37 44.45 0)
 			(hide yes)
@@
 			)
 		)
+		(property "LCSC" "C158012" (at 39.37 44.45 0) (hide yes) (effects (font (size 1 1))))
 	)
 	(symbol
@@
 			)
 		)
-		(property "MPN" "Generic 4.7uF X7R >=10V"
+		(property "MPN" "CL21B475KOFNNNE"
 			(at 64.77 82.55 0)
 			(hide yes)
@@
 			)
 		)
+		(property "LCSC" "C107365" (at 64.77 82.55 0) (hide yes) (effects (font (size 1 1))))
 	)
 	(symbol
@@
 			)
 		)
-		(property "MPN" "Generic 10uF X7R >=10V"
+		(property "MPN" "CL21B106KOQNNNE"
 			(at 240.03 124.46 0)
 			(hide yes)
@@
 			)
 		)
+		(property "LCSC" "C95841" (at 240.03 124.46 0) (hide yes) (effects (font (size 1 1))))
 	)
 	(symbol
@@
 			)
 		)
-		(property "MPN" "Generic 5.1k 1% 0603"
+		(property "MPN" "0603WAF5101T5E"
 			(at 90.17 179.07 0)
 			(hide yes)
@@
 			)
 		)
+		(property "LCSC" "C23186" (at 90.17 179.07 0) (hide yes) (effects (font (size 1 1))))
 	)
 	(symbol
@@
 			)
 		)
-		(property "MPN" "Generic 10k 1% 0603"
+		(property "MPN" "0603WAF1002T5E"
 			(at 309.88 154.94 0)
 			(hide yes)
@@
 			)
 		)
+		(property "LCSC" "C25804" (at 309.88 154.94 0) (hide yes) (effects (font (size 1 1))))
 	)
 	(symbol
@@
 			)
 		)
-		(property "MPN" "GCT USB4105-GF-A"
+		(property "MPN" "USB4105-GF-A-060"
 			(at 43.18 190.5 0)
 			(hide yes)
@@
 			)
 		)
+		(property "LCSC" "C3025063" (at 43.18 190.5 0) (hide yes) (effects (font (size 1 1))))
 	)
 	(symbol
@@
 			)
 		)
-		(property "MPN" "Generic 100nF X7R >=10V"
+		(property "MPN" "CC0603KRX7R9BB104"
 			(at 100.33 82.55 0)
 			(hide yes)
@@
 			)
 		)
+		(property "LCSC" "C14663" (at 100.33 82.55 0) (hide yes) (effects (font (size 1 1))))
 	)
 	(symbol
@@
 			)
 		)
-		(property "MPN" "E-Switch TL3342F160QG"
+		(property "MPN" "TS-1088-AR02016"
 			(at 350.52 154.94 0)
 			(hide yes)
@@
 			)
 		)
+		(property "LCSC" "C720477" (at 350.52 154.94 0) (hide yes) (effects (font (size 1 1))))
 	)
 	(symbol
@@
 			)
 		)
-		(property "MPN" "Generic 5.1k 1% 0603"
+		(property "MPN" "0603WAF5101T5E"
 			(at 90.17 208.28 0)
 			(hide yes)
@@
 			)
 		)
+		(property "LCSC" "C23186" (at 90.17 208.28 0) (hide yes) (effects (font (size 1 1))))
 	)
 	(symbol
@@
 			)
 		)
-		(property "MPN" "22uF 10V solid tantalum, case B"
+		(property "MPN" "TAJB226K010RNJ"
 			(at 144.78 82.55 0)
 			(hide yes)
@@
 			)
 		)
+		(property "LCSC" "C7198" (at 144.78 82.55 0) (hide yes) (effects (font (size 1 1))))
 	)
 	(symbol
@@
 			)
 		)
-		(property "MPN" "Generic 10k 1% 0603"
+		(property "MPN" "0603WAF1002T5E"
 			(at 350.52 124.46 0)
 			(hide yes)
@@
 			)
 		)
+		(property "LCSC" "C25804" (at 350.52 124.46 0) (hide yes) (effects (font (size 1 1))))
 	)
 	(symbol
@@
 			)
 		)
-		(property "MPN" "Generic 10k 1% 0603"
+		(property "MPN" "0603WAF1002T5E"
 			(at 234.95 72.39 0)
 			(hide yes)
@@
 			)
 		)
+		(property "LCSC" "C25804" (at 234.95 72.39 0) (hide yes) (effects (font (size 1 1))))
 	)
 	(symbol
@@
 			)
 		)
+		(property "LCSC" "C1855726" (at 224.79 219.71 0) (hide yes) (effects (font (size 1 1))))
 	)
 	(symbol
@@
 			)
 		)
-		(property "MPN" "Generic 10k 1% 0603"
+		(property "MPN" "0603WAF1002T5E"
 			(at 279.4 154.94 0)
 			(hide yes)
@@
 			)
 		)
+		(property "LCSC" "C25804" (at 279.4 154.94 0) (hide yes) (effects (font (size 1 1))))
 	)
 	(symbol
@@
 			)
 		)
+		(property "LCSC" "C6186" (at 105.41 44.45 0) (hide yes) (effects (font (size 1 1))))
 	)
 	(symbol
@@
 			)
 		)
-		(property "MPN" "Generic 22 1% 0603"
+		(property "MPN" "0603WAF220JT5E"
 			(at 154.94 185.42 90)
 			(hide yes)
@@
 			)
 		)
+		(property "LCSC" "C23345" (at 154.94 185.42 0) (hide yes) (effects (font (size 1 1))))
 	)
 	(symbol
@@
 			)
 		)
-		(property "MPN" "E-Switch TL3342F160QG"
+		(property "MPN" "TS-1088-AR02016"
 			(at 234.95 91.44 0)
 			(hide yes)
@@
 			)
 		)
+		(property "LCSC" "C720477" (at 234.95 91.44 0) (hide yes) (effects (font (size 1 1))))
 	)
 	(symbol
@@
 			)
 		)
-		(property "MPN" "Generic 22 1% 0603"
+		(property "MPN" "0603WAF220JT5E"
 			(at 154.94 214.63 90)
 			(hide yes)
@@
 			)
 		)
+		(property "LCSC" "C23345" (at 154.94 214.63 0) (hide yes) (effects (font (size 1 1))))
 	)
 	(symbol
@@
 			)
 		)
-		(property "MPN" "Generic 100nF X7R >=10V"
+		(property "MPN" "CC0603KRX7R9BB104"
 			(at 275.59 124.46 0)
 			(hide yes)
@@
 			)
 		)
+		(property "LCSC" "C14663" (at 275.59 124.46 0) (hide yes) (effects (font (size 1 1))))
 	)
 	(sheet
@@
 	)
 	(embedded_fonts no)
+	(wire (pts (xy 325.12 77.47) (xy 330.2 77.47)) (stroke (width 0) (type default)))
+	(label "STATUS_LED" (at 330.2 77.47 0) (effects (font (size 1.0 1.0)) (justify left bottom)))
+	(wire (pts (xy 265.43 220.98) (xy 265.43 215.9)) (stroke (width 0) (type default)))
+	(label "STATUS_LED" (at 265.43 215.9 0) (effects (font (size 1.0 1.0)) (justify left bottom)))
+	(wire (pts (xy 265.43 228.6) (xy 265.43 233.68)) (stroke (width 0) (type default)))
+	(label "STATUS_LED_A" (at 265.43 233.68 0) (effects (font (size 1.0 1.0)) (justify left bottom)))
+	(symbol (lib_id "Device:R") (at 265.43 224.79 0) (unit 1) (exclude_from_sim no) (in_bom yes) (on_board yes) (dnp no) (property "Reference" "R25" (at 270.43 222.79 0) (effects (font (size 1.1 1.1)) (justify left))) (property "Value" "1k" (at 270.43 225.79 0) (effects (font (size 1.0 1.0)) (justify left))) (property "Footprint" "Resistor_SMD:R_0603_1608Metric" (at 265.43 224.79 0) (effects (font (size 1.0 1.0)) (justify left)) (hide yes)) (property "Datasheet" "" (at 265.43 224.79 0) (effects (font (size 1.0 1.0)) (justify left)) (hide yes)) (property "Description" "Resistor" (at 265.43 224.79 0) (effects (font (size 1.0 1.0)) (justify left)) (hide yes)) (property "MPN" "0603WAF1001T5E" (at 265.43 224.79 0) (effects (font (size 1.0 1.0)) (justify left)) (hide yes)) (pin "1") (pin "2") (instances (project "sensors" (path "/655ba0f3-0427-5cf4-88d9-0bb38b1023d4" (reference "R25") (unit 1))))
+		(property "LCSC" "C21190" (at 265.43 224.79 0) (hide yes) (effects (font (size 1 1))))
+	)
+	(wire (pts (xy 265.43 254.0) (xy 265.43 259.08)) (stroke (width 0) (type default)))
+	(global_label "GND" (shape bidirectional) (at 265.43 259.08 0) (effects (font (size 1.0 1.0)) (justify left)) (property "Intersheetrefs" "${INTERSHEET_REFS}" (at 265.43 259.08 0) (hide yes) (effects (font (size 1.0 1.0)))))
+	(wire (pts (xy 265.43 246.38) (xy 265.43 241.3)) (stroke (width 0) (type default)))
+	(label "STATUS_LED_A" (at 265.43 241.3 0) (effects (font (size 1.0 1.0)) (justify left bottom)))
+	(symbol (lib_id "Device:LED") (at 265.43 250.19 90) (unit 1) (exclude_from_sim no) (in_bom yes) (on_board yes) (dnp no) (property "Reference" "D2" (at 278 247 0) (effects (font (size 1.1 1.1)) (justify left))) (property "Value" "GREEN / STATUS" (at 283 250 0) (effects (font (size 1.0 1.0)) (justify left))) (property "Footprint" "LED_SMD:LED_0603_1608Metric" (at 265.43 250.19 0) (effects (font (size 1.0 1.0))) (hide yes)) (property "Datasheet" "" (at 265.43 250.19 0) (effects (font (size 1.0 1.0))) (hide yes)) (property "Description" "Green status LED, pin 1 cathode to GND" (at 265.43 250.19 0) (effects (font (size 1.0 1.0))) (hide yes)) (property "MPN" "KT-0603YG" (at 265.43 250.19 0) (effects (font (size 1.0 1.0))) (hide yes)) (pin "1") (pin "2") (instances (project "sensors" (path "/655ba0f3-0427-5cf4-88d9-0bb38b1023d4" (reference "D2") (unit 1))))
+		(property "LCSC" "C2289" (at 265.43 250.19 0) (hide yes) (effects (font (size 1 1))))
+	)
+	(text "GPIO38 / pad34\nHIGH = LED on" (at 245 270 0) (effects (font (size 1.1 1.1)) (justify left top)))
 )

Commit message: Add Grove I2C passthrough board and update sensors manufacturing
Connections:
- net STATUS_LED: now also U1.31 (IO35); no longer U1.34 (IO38)
