File: pcb/sensors/sensors.kicad_sch (KiCad schematic)
At the start: 4 parts, among them J1 5V POWER, U1 XIAO ESP32-S3 / SOCKETED

Commit message: Route the sensors board and add the accontrol and pressure inputs
Finish the sensors PCB routing. Give the XIAO a local footprint that keeps
only the header holes (1.0 mm drill) with one courtyard per header, so parts
can sit under the module.

Add J9 (XH 5, accontrol J1 order) with ZC on GPIO1 and DIM_CMD on GPIO3, and
an optional ADS1115 (U6, 0x49) with J10 and the screen_sensors pressure
filter. Record why the CAN terminator R12 is a 1206.

Co-Authored-By: Claude Opus 5.5 <noreply@anthropic.com>
Parts:
- added C13, C15: 100nF, Capacitor_SMD:C_0603_1608Metric, symbol Device:C
- added C14: 10uF, Capacitor_SMD:C_0603_1608Metric, symbol Device:C
- added J10: PRESSURE, Connector_JST:JST_XH_B3B-XH-A_1x03_P2.50mm_Vertical, symbol Connector_Generic:Conn_01x03
- added R26: 1k, Resistor_SMD:R_0603_1608Metric, symbol Device:R
- added U6: ADS1115IDGSR, Package_SO:TSSOP-10_3x3mm_P0.5mm, symbol Analog_ADC:ADS1115IDGS
- U1: footprint Seeed_XIAO:XIAO-ESP32-S3-DIP -> Sensors_Local:XIAO-ESP32-S3-DIP-Headers
Connections:
- net +3V3: now also C13.1, C15.1, J10.1 (Pin_1), U6.1 (ADDR), U6.4 (AIN0), U6.8 (VDD)
- net GND: now also C13.2, C14.2, C15.2, J10.2 (Pin_2), U6.3 (GND)
- net I2C_SCL: now also U6.10 (SCL)
- net I2C_SDA: now also U6.9 (SDA)
- net ZC: now reaches U1.1 (D0)
- net DIM_CMD: now reaches U1.3 (D2)
- new net PRESSURE: J10.3 (Pin_3), R26.1
- new net PRESSURE_ADC: C14.1, R26.2, U6.5 (AIN1)
- no-connect marks 14 -> 15
Other:
- note added: "10. PRESSURE ADC - optional ADS1115, J10 = screen_sensors J3 order"
- note added: "Footprint: Sensors_Local:XIAO-ESP32-S3-DIP-Headers. Fit two female 1x7 sockets; XIAO fitted manually from stock. Row spacing 15.24mm; 2.54mm pitch. GPIO4 avoids boot straps."
- note added: "Seeed numbering: 1..7 = D0..D6; 8..11 = D7..D10. 12=3V3 OUT; 13=GND; 14=5V IN. Pins 15..25 are bottom pads, NC. D0/GPIO1 ZC input; D2/GPIO3 DIM_CMD output; D6/GPIO43 unused."
- note added: "U6 ADS1115 on the shared I2C bus, ADDR tied to 3V3: 0x49 (TMP102 already uses 0x48). A0 reads the local 3V3; A1 reads pressure through R26/C14 (1k / 10uF, 16 Hz, 10 ms). A2, A3 and ALERT/RDY unused. J10 pin order matches screen_sensors J3: same cable. XDB401 output 0.4-2.4V on 3V3 supply, not ratiometric: use the absolute A1 voltage."
- note removed: "Footprint: Seeed_XIAO:XIAO-ESP32-S3-DIP. Fit two female 1x7 sockets; XIAO fitted manually from stock. Row spacing 15.24mm; 2.54mm pitch. GPIO4 avoids boot straps."
- note removed: "Seeed numbering: 1..7 = D0..D6; 8..11 = D7..D10. 12=3V3 OUT; 13=GND; 14=5V IN. Pins 15..25 are bottom pads, NC. D0/GPIO1, D2/GPIO3 and D6/GPIO43 are unused."

Commit message: Swap ZC and DIM_CMD on the XIAO to ease routing
DIM_CMD moves to GPIO1 (pin 1) and ZC to GPIO3 (pin 3). GPIO3 only acts as
a strapping pin once STRAP_JTAG_SEL is burned, so the ZC level at reset is
harmless; accontrol's pull-down still keeps DIM low during boot.

Co-Authored-By: Claude Opus 5.5 <noreply@anthropic.com>
Connections:
- net DIM_CMD: now also U1.1 (D0); no longer U1.3 (D2)
- net ZC: now also U1.3 (D2); no longer U1.1 (D0)
Other:
- note added: "Seeed numbering: 1..7 = D0..D6; 8..11 = D7..D10. 12=3V3 OUT; 13=GND; 14=5V IN. Pins 15..25 are bottom pads, NC. D0/GPIO1 DIM_CMD output; D2/GPIO3 ZC input; D6/GPIO43 unused."
- note removed: "Seeed numbering: 1..7 = D0..D6; 8..11 = D7..D10. 12=3V3 OUT; 13=GND; 14=5V IN. Pins 15..25 are bottom pads, NC. D0/GPIO1 ZC input; D2/GPIO3 DIM_CMD output; D6/GPIO43 unused."
Changed lines of the file:
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@@
 (text "2. XIAO ESP32-S3 - two female 1x7 sockets, 2.54mm pitch" (at 180 15 0) (effects (font (size 1.7 1.7)) (justify left top)))
 (text "U1: D3/GPIO4 BOILER; D1/GPIO2 LED; D4/GPIO5 SDA; D5/GPIO6 SCL.\nD7/GPIO44 FLOW; D8/GPIO7 CAN TX; D9/GPIO8 CAN RX; D10/GPIO9 VALVE." (at 180 105 0) (effects (font (size 1.1 1.1)) (justify left top)))
-(text "Seeed numbering: 1..7 = D0..D6; 8..11 = D7..D10.\n12=3V3 OUT; 13=GND; 14=5V IN. Pins 15..25 are bottom pads, NC.\nD0/GPIO1 ZC input; D2/GPIO3 DIM_CMD output; D6/GPIO43 unused." (at 180 130 0) (effects (font (size 1.1 1.1)) (justify left top)))
+(text "Seeed numbering: 1..7 = D0..D6; 8..11 = D7..D10.\n12=3V3 OUT; 13=GND; 14=5V IN. Pins 15..25 are bottom pads, NC.\nD0/GPIO1 DIM_CMD output; D2/GPIO3 ZC input; D6/GPIO43 unused." (at 180 130 0) (effects (font (size 1.1 1.1)) (justify left top)))
 (text "Footprint: Sensors_Local:XIAO-ESP32-S3-DIP-Headers.\nFit two female 1x7 sockets; XIAO fitted manually from stock.\nRow spacing 15.24mm; 2.54mm pitch. GPIO4 avoids boot straps." (at 180 157 0) (effects (font (size 1.1 1.1)) (justify left top)))
 (text "3. STATUS LED - GPIO2 / D1, HIGH = ON" (at 18 179 0) (effects (font (size 1.7 1.7)) (justify left top)))
@@
 (embedded_fonts no)
 (wire (pts (xy 238.76 67.31) (xy 233.68 67.31)) (stroke (width 0) (type default)))
-(global_label "ZC" (shape bidirectional) (at 233.68 67.31 180) (effects (font (size 1.0 1.0)) (justify right)) (property "Intersheetrefs" "${INTERSHEET_REFS}" (at 233.68 67.31 180) (hide yes) (effects (font (size 1.0 1.0)))))
+(global_label "ZC" (shape bidirectional) (at 233.68 74.93 180) (effects (font (size 1.0 1.0)) (justify right)) (property "Intersheetrefs" "${INTERSHEET_REFS}" (at 233.68 74.93 180) (hide yes) (effects (font (size 1.0 1.0)))))
 (wire (pts (xy 238.76 71.12) (xy 233.68 71.12)) (stroke (width 0) (type default)))
 (global_label "HEATER_CMD" (shape bidirectional) (at 233.68 78.74 180) (effects (font (size 1.0 1.0)) (justify right)) (property "Intersheetrefs" "${INTERSHEET_REFS}" (at 233.68 78.74 180) (hide yes) (effects (font (size 1.0 1.0)))))
 (wire (pts (xy 238.76 74.93) (xy 233.68 74.93)) (stroke (width 0) (type default)))
-(global_label "DIM_CMD" (shape bidirectional) (at 233.68 74.93 180) (effects (font (size 1.0 1.0)) (justify right)) (property "Intersheetrefs" "${INTERSHEET_REFS}" (at 233.68 74.93 180) (hide yes) (effects (font (size 1.0 1.0)))))
+(global_label "DIM_CMD" (shape bidirectional) (at 233.68 67.31 180) (effects (font (size 1.0 1.0)) (justify right)) (property "Intersheetrefs" "${INTERSHEET_REFS}" (at 233.68 67.31 180) (hide yes) (effects (font (size 1.0 1.0)))))
 (wire (pts (xy 238.76 78.74) (xy 233.68 78.74)) (stroke (width 0) (type default)))
 (label "STATUS_LED" (at 233.68 71.12 0) (effects (font (size 1.0 1.0)) (justify right bottom)))

Commit message: Remove the accontrol connector J9 from the sensors board
The AC control board is shelved, so the valve and pump stay on the M5Stack
SSR (J7) and the RobotDyn dimmer (Grove I2C). Drop J9 and its wiring, and
leave D0/GPIO1 and D2/GPIO3 of the XIAO unconnected. The design notes say
how a future single AC board would take over from the dimmer I2C and J7.

The connectors now keep their J references on the PCB, hidden, with board
text labels for their functions.

Co-Authored-By: Claude Opus 5.5 <noreply@anthropic.com>
Connections:
- net DIM_CMD: no longer names the net of U1.1 (D0)
- net ZC: no longer names the net of U1.3 (D2)
- no-connect marks 15 -> 17
Other:
- note added: "Seeed numbering: 1..7 = D0..D6; 8..11 = D7..D10. 12=3V3 OUT; 13=GND; 14=5V IN. Pins 15..25 are bottom pads, NC. D0/GPIO1, D2/GPIO3 and D6/GPIO43 unused."
- note removed: "Seeed numbering: 1..7 = D0..D6; 8..11 = D7..D10. 12=3V3 OUT; 13=GND; 14=5V IN. Pins 15..25 are bottom pads, NC. D0/GPIO1 DIM_CMD output; D2/GPIO3 ZC input; D6/GPIO43 unused."
Changed lines of the file:
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@@
 (text "2. XIAO ESP32-S3 - two female 1x7 sockets, 2.54mm pitch" (at 180 15 0) (effects (font (size 1.7 1.7)) (justify left top)))
 (text "U1: D3/GPIO4 BOILER; D1/GPIO2 LED; D4/GPIO5 SDA; D5/GPIO6 SCL.\nD7/GPIO44 FLOW; D8/GPIO7 CAN TX; D9/GPIO8 CAN RX; D10/GPIO9 VALVE." (at 180 105 0) (effects (font (size 1.1 1.1)) (justify left top)))
-(text "Seeed numbering: 1..7 = D0..D6; 8..11 = D7..D10.\n12=3V3 OUT; 13=GND; 14=5V IN. Pins 15..25 are bottom pads, NC.\nD0/GPIO1 DIM_CMD output; D2/GPIO3 ZC input; D6/GPIO43 unused." (at 180 130 0) (effects (font (size 1.1 1.1)) (justify left top)))
+(text "Seeed numbering: 1..7 = D0..D6; 8..11 = D7..D10.\n12=3V3 OUT; 13=GND; 14=5V IN. Pins 15..25 are bottom pads, NC.\nD0/GPIO1, D2/GPIO3 and D6/GPIO43 unused." (at 180 130 0) (effects (font (size 1.1 1.1)) (justify left top)))
 (text "Footprint: Sensors_Local:XIAO-ESP32-S3-DIP-Headers.\nFit two female 1x7 sockets; XIAO fitted manually from stock.\nRow spacing 15.24mm; 2.54mm pitch. GPIO4 avoids boot straps." (at 180 157 0) (effects (font (size 1.1 1.1)) (justify left top)))
 (text "3. STATUS LED - GPIO2 / D1, HIGH = ON" (at 18 179 0) (effects (font (size 1.7 1.7)) (justify left top)))
@@
 (sheet_instances (path "/" (page "1")))
 (embedded_fonts no)
-(wire (pts (xy 238.76 67.31) (xy 233.68 67.31)) (stroke (width 0) (type default)))
-(global_label "ZC" (shape bidirectional) (at 233.68 74.93 180) (effects (font (size 1.0 1.0)) (justify right)) (property "Intersheetrefs" "${INTERSHEET_REFS}" (at 233.68 74.93 180) (hide yes) (effects (font (size 1.0 1.0)))))
 (wire (pts (xy 238.76 71.12) (xy 233.68 71.12)) (stroke (width 0) (type default)))
 (global_label "HEATER_CMD" (shape bidirectional) (at 233.68 78.74 180) (effects (font (size 1.0 1.0)) (justify right)) (property "Intersheetrefs" "${INTERSHEET_REFS}" (at 233.68 78.74 180) (hide yes) (effects (font (size 1.0 1.0)))))
-(wire (pts (xy 238.76 74.93) (xy 233.68 74.93)) (stroke (width 0) (type default)))
-(global_label "DIM_CMD" (shape bidirectional) (at 233.68 67.31 180) (effects (font (size 1.0 1.0)) (justify right)) (property "Intersheetrefs" "${INTERSHEET_REFS}" (at 233.68 67.31 180) (hide yes) (effects (font (size 1.0 1.0)))))
 (wire (pts (xy 238.76 78.74) (xy 233.68 78.74)) (stroke (width 0) (type default)))
 (label "STATUS_LED" (at 233.68 71.12 0) (effects (font (size 1.0 1.0)) (justify right bottom)))
@@
 (wire (pts (xy 238.76 86.36) (xy 233.68 86.36)) (stroke (width 0) (type default)))
 (global_label "I2C_SCL" (shape bidirectional) (at 233.68 86.36 180) (effects (font (size 1.0 1.0)) (justify right)) (property "Intersheetrefs" "${INTERSHEET_REFS}" (at 233.68 86.36 180) (hide yes) (effects (font (size 1.0 1.0)))))
+(no_connect (at 238.76 67.31))
+(no_connect (at 238.76 74.93))
 (no_connect (at 238.76 90.17))
 (wire (pts (xy 281.94 90.17) (xy 287.02 90.17)) (stroke (width 0) (type default)))
