File: pcb/accontrol/accontrol.kicad_sch (KiCad schematic)
At the start: 35 parts, among them J1 CTRL, J2 MAINS_IN, J3 VALVE, J4 PUMP, Q1 SS8050, Q2 BT136S-600E, Q3 SS8050, Q4 BT136S-600E, U1 MOC3043M, U2 MOC3023M, U3 EL817C

Commit message: Document the AC control board and pick its JLCPCB parts
Add the design notes for the AC control board: input stages, triac gate
drive, zero-cross pulse, pump firing rules and the overvoltage decision.
Drop the varistor across the valve triac and keep the 400 V optotriacs.

Put the ABS6 bridge on its 4 mm pitch footprint and fill the ABS6 and
BT136S parts from JLCPCB. Import the footprints into the PCB and add the
component datasheets.

Co-Authored-By: Claude Opus 5.5 <noreply@anthropic.com>
Parts:
- removed RV1: 430V, Resistor_SMD:R_1210_3225Metric, symbol Device:Varistor
- D3: footprint Package_TO_SOT_SMD:TO-269AA -> Diode_SMD:Diode_Bridge_Diotec_ABS; LCSC (none) -> C48642435; Note MDD ABS6, 600 V -> Hongjiacheng ABS6, 600 V, ABS package (4 mm pitch)
- Q2, Q4: value BT136S-600E -> BT136S; LCSC (none) -> C23427; MPN BT136S-600E -> BT136S
Changed lines of the file:
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@@
 (symbol (lib_id "Triac_Thyristor:BT136-600") (at 137.16 49.53 0) (unit 1) (exclude_from_sim no) (in_bom yes) (on_board yes) (dnp no)
   (property "Reference" "Q2" (at 141.605 48.26 0) (effects (font (size 1.27 1.27)) (justify left)))
-  (property "Value" "BT136S-600E" (at 141.605 50.8 0) (effects (font (size 1.27 1.27)) (justify left)))
+  (property "Value" "BT136S" (at 141.605 50.8 0) (effects (font (size 1.27 1.27)) (justify left)))
   (property "Footprint" "Package_TO_SOT_SMD:TO-252-2" (at 137.16 49.53 0) (effects (font (size 1.27 1.27))) (hide yes))
   (property "Datasheet" "" (at 137.16 49.53 0) (effects (font (size 1.27 1.27))) (hide yes))
-  (property "MPN" "BT136S-600E" (at 137.16 49.53 0) (effects (font (size 1.27 1.27))) (hide yes))
-  (property "LCSC" "" (at 137.16 49.53 0) (effects (font (size 1.27 1.27))) (hide yes))
+  (property "MPN" "BT136S" (at 137.16 49.53 0) (effects (font (size 1.27 1.27))) (hide yes))
+  (property "LCSC" "C23427" (at 137.16 49.53 0) (effects (font (size 1.27 1.27))) (hide yes))
   (property "Note" "DPAK: 1 MT1, 2 MT2 (tab), 3 G" (at 137.16 49.53 0) (effects (font (size 1.27 1.27))) (hide yes))
   (pin "1")
@@
 (junction (at 137.16 36.83) (diameter 0) (color 0 0 0 0))
 (junction (at 147.32 36.83) (diameter 0) (color 0 0 0 0))
-(junction (at 157.48 36.83) (diameter 0) (color 0 0 0 0))
 (wire (pts (xy 137.16 62.23) (xy 147.32 62.23)) (stroke (width 0) (type default)))
 (wire (pts (xy 147.32 62.23) (xy 157.48 62.23)) (stroke (width 0) (type default)))
@@
 (wire (pts (xy 147.32 59.69) (xy 147.32 62.23)) (stroke (width 0) (type default)))
 (junction (at 147.32 62.23) (diameter 0) (color 0 0 0 0))
-(junction (at 157.48 62.23) (diameter 0) (color 0 0 0 0))
-(symbol (lib_id "Device:Varistor") (at 157.48 49.53 0) (unit 1) (exclude_from_sim no) (in_bom yes) (on_board yes) (dnp no)
-  (property "Reference" "RV1" (at 160.01999999999998 48.26 0) (effects (font (size 1.27 1.27)) (justify left)))
-  (property "Value" "430V" (at 160.01999999999998 50.800000000000004 0) (effects (font (size 1.27 1.27)) (justify left)))
-  (property "Footprint" "Resistor_SMD:R_1210_3225Metric" (at 157.48 49.53 0) (effects (font (size 1.27 1.27))) (hide yes))
-  (property "Datasheet" "" (at 157.48 49.53 0) (effects (font (size 1.27 1.27))) (hide yes))
-  (property "MPN" "" (at 157.48 49.53 0) (effects (font (size 1.27 1.27))) (hide yes))
-  (property "LCSC" "" (at 157.48 49.53 0) (effects (font (size 1.27 1.27))) (hide yes))
-  (property "Note" "1210 MOV, 275 VAC (as M5Stack)" (at 157.48 49.53 0) (effects (font (size 1.27 1.27))) (hide yes))
-  (pin "1")
-  (pin "2")
-  (instances (project "accontrol" (path "/a3ee807d-f8aa-4db3-ad94-73a886b6ed37" (reference "RV1") (unit 1)))))
-(wire (pts (xy 157.48 36.83) (xy 157.48 45.72)) (stroke (width 0) (type default)))
-(wire (pts (xy 157.48 53.34) (xy 157.48 62.23)) (stroke (width 0) (type default)))
 (label "L" (at 167.64 36.83 0) (effects (font (size 1.27 1.27)) (justify left bottom)))
 (label "L_VALVE" (at 167.64 62.23 0) (effects (font (size 1.27 1.27)) (justify left bottom)))
@@
 (symbol (lib_id "Triac_Thyristor:BT136-600") (at 137.16 99.06 0) (unit 1) (exclude_from_sim no) (in_bom yes) (on_board yes) (dnp no)
   (property "Reference" "Q4" (at 141.605 97.79 0) (effects (font (size 1.27 1.27)) (justify left)))
-  (property "Value" "BT136S-600E" (at 141.605 100.33000000000001 0) (effects (font (size 1.27 1.27)) (justify left)))
+  (property "Value" "BT136S" (at 141.605 100.33000000000001 0) (effects (font (size 1.27 1.27)) (justify left)))
   (property "Footprint" "Package_TO_SOT_SMD:TO-252-2" (at 137.16 99.06 0) (effects (font (size 1.27 1.27))) (hide yes))
   (property "Datasheet" "" (at 137.16 99.06 0) (effects (font (size 1.27 1.27))) (hide yes))
-  (property "MPN" "BT136S-600E" (at 137.16 99.06 0) (effects (font (size 1.27 1.27))) (hide yes))
-  (property "LCSC" "" (at 137.16 99.06 0) (effects (font (size 1.27 1.27))) (hide yes))
+  (property "MPN" "BT136S" (at 137.16 99.06 0) (effects (font (size 1.27 1.27))) (hide yes))
+  (property "LCSC" "C23427" (at 137.16 99.06 0) (effects (font (size 1.27 1.27))) (hide yes))
   (property "Note" "DPAK: 1 MT1, 2 MT2 (tab), 3 G" (at 137.16 99.06 0) (effects (font (size 1.27 1.27))) (hide yes))
   (pin "1")
@@
   (property "Reference" "D3" (at 137.16 143.51 90) (effects (font (size 1.27 1.27)) (justify left)))
   (property "Value" "ABS6" (at 137.16 161.29000000000002 90) (effects (font (size 1.27 1.27)) (justify left)))
-  (property "Footprint" "Package_TO_SOT_SMD:TO-269AA" (at 132.07999999999998 152.4 90) (effects (font (size 1.27 1.27))) (hide yes))
+  (property "Footprint" "Diode_SMD:Diode_Bridge_Diotec_ABS" (at 132.07999999999998 152.4 90) (effects (font (size 1.27 1.27))) (hide yes))
   (property "Datasheet" "" (at 132.07999999999998 152.4 90) (effects (font (size 1.27 1.27))) (hide yes))
   (property "MPN" "ABS6" (at 132.07999999999998 152.4 90) (effects (font (size 1.27 1.27))) (hide yes))
-  (property "LCSC" "" (at 132.07999999999998 152.4 90) (effects (font (size 1.27 1.27))) (hide yes))
-  (property "Note" "MDD ABS6, 600 V" (at 132.07999999999998 152.4 90) (effects (font (size 1.27 1.27))) (hide yes))
-  (pin "1")
-  (pin "2")
+  (property "LCSC" "C48642435" (at 132.07999999999998 152.4 90) (effects (font (size 1.27 1.27))) (hide yes))
+  (property "Note" "Hongjiacheng ABS6, 600 V, ABS package (4 mm pitch)" (at 132.07999999999998 152.4 90) (effects (font (size 1.27 1.27))) (hide yes))
+  (pin "1")
+  (pin "2")

Commit message: Shelve the AC control board with its layout study
The machine keeps the RobotDyn dimmer and the M5Stack Unit SSR. A single
board with both channels, the zero-cross sense and the fuse needs about
80 x 30 mm, while the AC enclosure offers 68 x 31.6 mm inside, and the
single cable it would bring did not justify a home-made 230 V board.

Keep the work as a reference: AC and Mains net classes with DRC rules for
2.5 mm between mains nets and 7 mm to the 3V3 side, slotted optocoupler
footprints, HT396R right-angle headers, an AEM 2410 fuse (100 A breaking),
1210 resistors for the zero-cross divider and the pump snubber, L_IN
between J2 and F1, and the partial valve-channel layout.

Co-Authored-By: Claude Opus 5.5 <noreply@anthropic.com>
Parts:
- F1: footprint Fuse:Fuse_2512_6332Metric -> Accontrol_Local:F2410; LCSC (none) -> C83797; MPN 2410 2A 250V fast -> MF2410F2.000TM; Note Check footprint against the chosen 2410 fuse -> AEM 2410 fast, 100 A breaking at 250 VAC
- J1: Note 1 GND, 2 3V3, 3 ZC, 4 DIM, 5 SSR -> 1 GND, 2 3V3, 3 DIM, 4 ZC, 5 SSR
- J2, J3, J4: footprint Connector_JST:JST_VH_B2P-VH_1x02_P3.96mm_Vertical -> Accontrol_Local:CONN-TH_P3.96_HT396R-3.96-2P; LCSC (none) -> C577799; MPN HT3.96-2P -> HT396R-3.96-2P
- R13: footprint Resistor_SMD:R_1206_3216Metric -> Resistor_SMD:R_1210_3225Metric; LCSC (none) -> C728404; MPN (none) -> RC1210JR-0739RL; Note Snubber -> Snubber, 1210 for the C3 discharge at each firing
- R14: footprint Resistor_SMD:R_1206_3216Metric -> Resistor_SMD:R_1210_3225Metric; LCSC (none) -> C422421; MPN (none) -> 1210W2F1203T5E; Note ZC sense, 2 x 120k in series = 240k: 0.11 W and 160 V peak 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 -> ZC sense, 2 x 120k 1210 in series = 240k: 0.11 W (22 %) and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
- R15: footprint Resistor_SMD:R_1206_3216Metric -> Resistor_SMD:R_1210_3225Metric; LCSC (none) -> C422421; MPN (none) -> 1210W2F1203T5E
- U1, U2: footprint Package_DIP:SMDIP-6_W9.53mm -> Accontrol_Local:SMDIP-6_W9.53mm_Slot
- U3: footprint Package_DIP:SMDIP-4_W9.53mm -> Accontrol_Local:SMDIP-4_W9.53mm_Slot
Connections:
- net DIM: now also J1.3 (Pin_3); no longer J1.4 (Pin_4)
- net ZC: now also J1.4 (Pin_4); no longer J1.3 (Pin_3)
- net L_IN: now reaches F1.2, J2.1 (Pin_1)
