File: pcb/i2cterm/i2cterm.kicad_pcb (KiCad board)
At the start: 2 copper layers, 17.5 x 20 mm, 8 parts, among them J1 GROVE VERTICAL, J2 GROVE VERTICAL

Commit message: Use the basic-library red LED C2286 on the i2cterm board
D1 moves from the extended KT-0603YG green LED (C2289) to the KT-0603R red
LED (C2286), a JLCPCB basic part from the same KENTO 0603 family, which
avoids the extended-part fee. The footprint and the 1k resistor stay; the
current rises from about 1.2 to 1.4 mA. The JLCPCB assembly preview shows
the cathode on the GND pad.

Co-Authored-By: Claude Opus 5.5 <noreply@anthropic.com>
Parts:
- D1: value GREEN -> RED
Changed lines of the file:
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@@
 			)
 		)
-		(property "Value" "GREEN"
+		(property "Value" "RED"
 			(at 0.674448 -1.313482 270)
 			(layer "F.Fab")
@@
 			)
 		)
-		(property "MPN" "KT-0603YG"
+		(property "MPN" "KT-0603R"
 			(at 0 0 270)
 			(layer "F.Fab")
@@
 			)
 		)
-		(property "LCSC" "C2289"
+		(property "LCSC" "C2286"
 			(at 0 0 0)
 			(layer "F.Fab")
