File: pcb/combined/combined.kicad_sch (KiCad schematic)
At the start: 27 parts, among them J2 MAINS_IN, J3 VALVE, J9 PUMP, Q1 SS8050, Q2 BT136S, U1 MOC3043M, U8 EL817C, U9 EL817C

Commit message: Move combined to basic passives, M2 holes and an HT3.96 flow connector
- Mounting holes H1 to H6 become M2 (2.2 mm NPTH) and move on the board;
  the AC wing narrows to 35 mm.
- Nine extended passives become JLCPCB basic parts: R3 150, R5/R6
  300 + 300, R7 100 (1206 kept: an 0805 breaks the 1.5 mm L-side
  clearance), FB divider 120k/30k (5.00 V), EN divider 330k/24k
  (18.2 V / 16.7 V), C1 10 uF 1206, C5 220 nF 0805, setpoint filter
  1.5k / 2.2 uF. Only C2 (10 nF 1 kV) stays extended.
- J6 (flow) becomes a Kefa HT396V-3.96-3P: the Digmesa 0.5 mm2 wires
  screw into the plug without the JST-SM to XH adapter. Footprint and
  3D model from LCSC, checked against the Kefa drawing.
- The MPB003 manufacturer datasheet replaces gearpump.pdf; it confirms
  the 7-wire pinout used on J9.

Co-Authored-By: Claude Opus 5.5 <noreply@anthropic.com>
Parts:
- C20, C21: value 1.5uF -> 2.2uF; LCSC C384767 -> C377773; MPN 0805B155K250CT -> CL21A225KBQNNNE; Note Setpoint filter, 25 V X7R -> Setpoint filter, 50 V X5R
- R3: value 180 -> 150; LCSC C22828 -> C22808; MPN 0603WAF1800T5E -> 0603WAF1500T5E; Note MOC LED: (3.3-1.2-0.1)/180 = 11 mA typ, >= 8 mA worst case -> MOC LED: (3.3-1.2-0.1)/150 = 13 mA typ, >= 9.6 mA worst case
- R36, R37: value 2.2k -> 1.5k; LCSC C4190 -> C22843; MPN 0603WAF2201T5E -> 0603WAF1501T5E
- R5: value 360 -> 300; LCSC C163378 -> C17887; MPN RC1206FR-07360RL -> 1206W4F3000T5E; Note MT2 series resistor (M5Stack design) -> MT2 series resistor; R5 + R6 = 600 ohms
- R6: value 330 -> 300; LCSC C17930 -> C17887; MPN 1206W4F3300T5E -> 1206W4F3000T5E; Note Gate series resistor (M5Stack design) -> Gate series resistor; R5 + R6 = 600 ohms
- R7: value 39 -> 100; LCSC C22198 -> C17901; MPN 1206W4F390JT5E -> 1206W4F1000T5E
Other:
- note added: "GND_P, +5V_P, SPEED_P and TACHO_P belong to the pump (green, yellow, brown, blue wires): never tie them to board GND or +5V. Rotation (white) stays unconnected in the cable. U8 off (reset, boot, XIAO absent): R35 pulls the setpoint to GND_P, pump stopped. PWM 1 kHz, 16 bits on GPIO1; 2 x 1.5k / 2.2uF filter: 48 Hz, about 12 mV ripple, 10 ms response. PUMP_TACHO is low while blue is low; count its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"
- note removed: "GND_P, +5V_P, SPEED_P and TACHO_P belong to the pump (green, yellow, brown, blue wires): never tie them to board GND or +5V. Rotation (white) stays unconnected in the cable. U8 off (reset, boot, XIAO absent): R35 pulls the setpoint to GND_P, pump stopped. PWM 1 kHz, 16 bits on GPIO1; 2 x 2.2k / 1.5uF filter: 48 Hz, about 12 mV ripple, 10 ms response. PUMP_TACHO is low while blue is low; count its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"
Changed lines of the file:
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@@
 			)
 		)
-		(property "Value" "39"
+		(property "Value" "100"
 			(at 149.86 45.72 0)
 			(show_name no)
@@
 			)
 		)
-		(property "MPN" "1206W4F390JT5E"
+		(property "MPN" "1206W4F1000T5E"
 			(at 147.32 44.45 0)
 			(hide yes)
@@
 			)
 		)
-		(property "LCSC" "C22198"
+		(property "LCSC" "C17901"
 			(at 147.32 44.45 0)
 			(hide yes)
@@
 			)
 		)
-		(property "Value" "360"
+		(property "Value" "300"
 			(at 125.73 44.704 90)
 			(show_name no)
@@
 			)
 		)
-		(property "MPN" "RC1206FR-07360RL"
+		(property "MPN" "1206W4F3000T5E"
 			(at 125.73 46.99 90)
 			(hide yes)
@@
 			)
 		)
-		(property "LCSC" "C163378"
+		(property "LCSC" "C17887"
 			(at 125.73 46.99 90)
 			(hide yes)
@@
 			)
 		)
-		(property "Note" "MT2 series resistor (M5Stack design)"
+		(property "Note" "MT2 series resistor; R5 + R6 = 600 ohms"
 			(at 125.73 46.99 90)
 			(hide yes)
@@
 			)
 		)
-		(property "Value" "180"
+		(property "Value" "150"
 			(at 100.33 49.53 90)
 			(show_name no)
@@
 			)
 		)
-		(property "MPN" "0603WAF1800T5E"
+		(property "MPN" "0603WAF1500T5E"
 			(at 100.33 46.99 90)
 			(hide yes)
@@
 			)
 		)
-		(property "LCSC" "C22828"
+		(property "LCSC" "C22808"
 			(at 100.33 46.99 90)
 			(hide yes)
@@
 			)
 		)
-		(property "Note" "MOC LED: (3.3-1.2-0.1)/180 = 11 mA typ, >= 8 mA worst case"
+		(property "Note" "MOC LED: (3.3-1.2-0.1)/150 = 13 mA typ, >= 9.6 mA worst case"
 			(at 100.33 46.99 90)
 			(hide yes)
@@
 			)
 		)
-		(property "Value" "330"
+		(property "Value" "300"
 			(at 125.73 56.642 90)
 			(show_name no)
@@
 			)
 		)
-		(property "MPN" "1206W4F3300T5E"
+		(property "MPN" "1206W4F3000T5E"
 			(at 125.73 52.07 90)
 			(hide yes)
@@
 			)
 		)
-		(property "LCSC" "C17930"
+		(property "LCSC" "C17887"
 			(at 125.73 52.07 90)
 			(hide yes)
@@
 			)
 		)
-		(property "Note" "Gate series resistor (M5Stack design)"
+		(property "Note" "Gate series resistor; R5 + R6 = 600 ohms"
 			(at 125.73 52.07 90)
 			(hide yes)
@@
 			)
 		)
-		(property "Value" "2.2k"
+		(property "Value" "1.5k"
 			(at 109.22 104.394 90)
 			(show_name no)
@@
 			)
 		)
-		(property "MPN" "0603WAF2201T5E"
+		(property "MPN" "0603WAF1501T5E"
 			(at 109.22 106.68 90)
 			(hide yes)
@@
 			)
 		)
-		(property "LCSC" "C4190"
+		(property "LCSC" "C22843"
 			(at 109.22 106.68 90)
 			(hide yes)
@@
 			)
 		)
-		(property "Value" "1.5uF"
+		(property "Value" "2.2uF"
 			(at 119.38 111.76 0)
 			(show_name no)
@@
 			)
 		)
-		(property "MPN" "0805B155K250CT"
+		(property "MPN" "CL21A225KBQNNNE"
 			(at 116.84 110.49 0)
 			(hide yes)
@@
 			)
 		)
-		(property "LCSC" "C384767"
+		(property "LCSC" "C377773"
 			(at 116.84 110.49 0)
 			(hide yes)
@@
 			)
 		)
-		(property "Note" "Setpoint filter, 25 V X7R"
+		(property "Note" "Setpoint filter, 50 V X5R"
 			(at 116.84 110.49 0)
 			(hide yes)
@@
 			)
 		)
-		(property "Value" "2.2k"
+		(property "Value" "1.5k"
 			(at 124.46 104.394 90)
 			(show_name no)
@@
 			)
 		)
-		(property "MPN" "0603WAF2201T5E"
+		(property "MPN" "0603WAF1501T5E"
 			(at 124.46 106.68 90)
 			(hide yes)
@@
 			)
 		)
-		(property "LCSC" "C4190"
+		(property "LCSC" "C22843"
 			(at 124.46 106.68 90)
 			(hide yes)
@@
 			)
 		)
-		(property "Value" "1.5uF"
+		(property "Value" "2.2uF"
 			(at 134.62 111.76 0)
 			(show_name no)
@@
 			)
 		)
-		(property "MPN" "0805B155K250CT"
+		(property "MPN" "CL21A225KBQNNNE"
 			(at 132.08 110.49 0)
 			(hide yes)
@@
 			)
 		)
-		(property "LCSC" "C384767"
+		(property "LCSC" "C377773"
 			(at 132.08 110.49 0)
 			(hide yes)
@@
 			)
 		)
-		(property "Note" "Setpoint filter, 25 V X7R"
+		(property "Note" "Setpoint filter, 50 V X5R"
 			(at 132.08 110.49 0)
 			(hide yes)
@@
 		)
 	)
-	(text "GND_P, +5V_P, SPEED_P and TACHO_P belong to the pump (green, yellow, brown, blue wires):\nnever tie them to board GND or +5V. Rotation (white) stays unconnected in the cable.\nU8 off (reset, boot, XIAO absent): R35 pulls the setpoint to GND_P, pump stopped.\nPWM 1 kHz, 16 bits on GPIO1; 2 x 2.2k / 1.5uF filter: 48 Hz, about 12 mV ripple, 10 ms response.\nPUMP_TACHO is low while blue is low; count its edges (PCNT)."
+	(text "GND_P, +5V_P, SPEED_P and TACHO_P belong to the pump (green, yellow, brown, blue wires):\nnever tie them to board GND or +5V. Rotation (white) stays unconnected in the cable.\nU8 off (reset, boot, XIAO absent): R35 pulls the setpoint to GND_P, pump stopped.\nPWM 1 kHz, 16 bits on GPIO1; 2 x 1.5k / 2.2uF filter: 48 Hz, about 12 mV ripple, 10 ms response.\nPUMP_TACHO is low while blue is low; count its edges (PCNT)."
 		(exclude_from_sim no)
 		(at 20 158 0)
