File: pcb/combined/combined_controller.kicad_sch (KiCad schematic)
At the start: 13 parts, among them J1 5V POWER, J10 PRESSURE, J11 XIAO D0-D6, J12 XIAO D7-5V, U6 ADS1115IDGSR, U7 XIAO ESP32-S3 / SOCKETED

Commit message: Route the combined board to a clean DRC and export it for JLCPCB
Rules follow IEC 60335-1 for functional insulation: 2.2 mm between mains
nets, 1.5 mm or 1.1 mm between mains nets a few volts apart, and the
track-into-pad exception tied to the part a track enters. The HT3.96
connectors get oval pads, the datasheet's 1.6 mm holes and a milled slot
between L and N. C2/C3 move to 1812, R12 splits into R12 + R27, and every
part has its JLCPCB number. The exporter accepts polygon outlines, and the
placement corrections come from the supplier footprints. H2 and H3 are
added to the schematic.

Co-Authored-By: Claude Opus 5.5 <noreply@anthropic.com>
Parts:
- added H2, H3: M2.5, MountingHole:MountingHole_2.7mm_M2.5, symbol Mechanical:MountingHole
- D4: value GREEN / STATUS -> STATUS; footprint LED_SMD:LED_0805_2012Metric -> LED_SMD:LED_0603_1608Metric; LCSC C2297 -> C2286; MPN KT-0805G -> KT-0603R
Other:
- note added: "H1, H2, H3: M2.5 mounting holes, 2.7mm NPTH, not connected. H2 sits on the mains side: nylon screw and standoff, at least 5 mm tall."
- note removed: "H1: M2.5 mounting hole, 2.7mm NPTH, not connected."

Commit message: Draw the combined v2 schematic: 24 V buck and isolated gear pump interface
The pump dimmer and the zero-cross detector leave the board; the 230 V
valve channel stays. J7 brings 24 V from the pump supply to an
LMR33630A buck (5.02 V, enable at 18.4 V, off at 16.9 V), and J1 now sends
5 V to the screen. Two EL817C keep the pump's signal wires on their
isolated side: U8 turns the 1 kHz PWM on GPIO1 into a filtered setpoint
from the pump's own 5 V, U9 brings the tachometer back to GPIO3. DIM and
ZC become PUMP_SPEED and PUMP_TACHO.

The XIAO 5V pin is its USB VBUS with no diode; no diode is added either,
so USB is never plugged in with the XIAO on the board. New parts take new
references, so that no low-voltage net inherits a stale Mains netclass
pattern; those patterns and the pump and zero-cross DRC rules are gone.

F1 drops to 0.5 A, now that it protects the valve alone, and the AC
tracks to 1 mm. J3 is reversed so that its N faces N on J2. The HT396R
outline follows the Kefa drawing, and J8 becomes an HT396V header whose
screw plug takes the 0.75 mm² wires to the boiler SSR.

The board has been updated from the schematic; placement and routing are
still in progress.

Co-Authored-By: Claude Opus 5.5 <noreply@anthropic.com>
Parts:
- added C1, C4: 10uF 50V, Capacitor_SMD:C_1210_3225Metric, symbol Device:C
- added C16: 1uF, Capacitor_SMD:C_0603_1608Metric, symbol Device:C
- added C17, C18, C19: 22uF, Capacitor_SMD:C_1206_3216Metric, symbol Device:C
- added C5, C7: 100nF, Capacitor_SMD:C_0603_1608Metric, symbol Device:C
- added C6: 47uF 50V, Capacitor_SMD:CP_Elec_6.3x7.7, symbol Device:C_Polarized
- added D5: 5V, LED_SMD:LED_0603_1608Metric, symbol Device:LED
- added J7: 24V IN, Combined_Local:CONN-TH_P3.96_HT396R-3.96-2P, symbol Connector_Generic:Conn_01x02
- added L1: 10uH, Inductor_SMD:L_Changjiang_FXL0630, symbol Device:L
- added R28, R30: 100k, Resistor_SMD:R_0603_1608Metric, symbol Device:R
- added R29: 24.9k, Resistor_SMD:R_0603_1608Metric, symbol Device:R
- added R31: 7.15k, Resistor_SMD:R_0603_1608Metric, symbol Device:R
- added R32: 1k, Resistor_SMD:R_0603_1608Metric, symbol Device:R
- added U10: LMR33630ADDAR, Package_SO:Texas_HSOP-8-1EP_3.9x4.9mm_P1.27mm_ThermalVias, symbol Regulator_Switching:LMR33630ADDA
- J1: value 5V POWER -> 5V SCREEN
Connections:
- net +5V: now also C17.1, C18.1, C19.1, L1.2, R28.1, R32.1
- net GND: now also C1.2, C16.2, C17.2, C18.2, C19.2, C4.2, C5.2, C6.2, D5.1 (K), J7.1 (Pin_1), R29.2, R31.2, U10.1 (GND), U10.9 (GND)
- net DIM renamed PUMP_SPEED
- net ZC renamed PUMP_TACHO
- new net: D5.2 (A), R32.2
- new net: R28.2, R29.1, U10.5 (FB)
- new net: C16.1, U10.6 (VCC)
- new net: R30.2, R31.1, U10.3 (EN)
- new net: C7.2, L1.1, U10.8 (SW)
- new net: C7.1, U10.7 (BOOT)
- new net +24V: C1.1, C4.1, C5.1, C6.1, J7.2 (Pin_2), R30.1, U10.2 (VIN)
- no-connect marks 16 -> 17
Other:
- note added: "1. POWER - 24 V in (J7), 24 to 5 V buck (U10), 5 V out to the screen (J1), XIAO 3.3 V regulator"
- note added: "U10 LMR33630A, 400 kHz: 5.02 V with R28/R29 (100k / 24.9k). EN divider R30/R31 (100k / 7.15k): starts at 18.4 V, stops at 16.9 V. +5V feeds J1 (screen), CAN, FLOW and the boiler SSR output. The XIAO 5V pin is VBUS of its USB-C, with no diode: never plug USB into the XIAO on this board. USB would drive +5V and, through the buck high-side body diode, the 24 V rail. Flash it off the board. XIAO 3V3 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"
- note added: "U7: D0/GPIO1 PUMP_SPEED; D1/GPIO2 LED; D2/GPIO3 PUMP_TACHO; D3/GPIO4 BOILER. D4/GPIO5 SDA; D5/GPIO6 SCL; D7/GPIO44 FLOW; D8/GPIO7 CAN TX. D9/GPIO8 CAN RX; D10/GPIO9 SSR (valve)."
- note removed: "1. POWER - external regulated 5V / XIAO onboard 3.3V regulator"
- note removed: "J1 feeds XIAO 5V and the 5V interfaces. XIAO 3V3 supplies CAN VIO, I2C, TMP102, ADS1115, FLOW pull-up and the AC-side logic (SSR/DIM drivers, ZC pull-up). USB-C, LDO, BOOT and RESET are on the removable XIAO. Disconnect external J1 power before USB flashing."
- note removed: "U7: D0/GPIO1 DIM; D1/GPIO2 LED; D2/GPIO3 ZC; D3/GPIO4 BOILER. D4/GPIO5 SDA; D5/GPIO6 SCL; D7/GPIO44 FLOW; D8/GPIO7 CAN TX. D9/GPIO8 CAN RX; D10/GPIO9 SSR (valve)."
- moved on the sheet: J1

Commit message: Route combined v2: buck layout, POWER class with GND, GPIO table on the back
Shrink F.Fab texts to 0.5 mm and silkscreen texts to 0.8 mm. Put GND in
the POWER net class and enforce its 0.3 mm minimum by a DRC rule, with a
0.2 mm neck-down allowed at the TMP102. Add the XIAO GPIO table on
B.SilkS and the 24 V and 230 V ratings.

Swap R5 to C163378 and U6 to ADS1115IDGST (C468683), same parts in stock.
Fix the JLCPCB placement of U5 (+270) and J9 (pin-row midpoint, +180).

Co-Authored-By: Claude Opus 5.5 <noreply@anthropic.com>
Parts:
- removed C4: 10uF 50V, Capacitor_SMD:C_1210_3225Metric, symbol Device:C
- removed C6: 47uF 50V, Capacitor_SMD:CP_Elec_6.3x7.7, symbol Device:C_Polarized
- added H4, H5: M2.5, MountingHole:MountingHole_2.7mm_M2.5, symbol Mechanical:MountingHole
- C5: value 100nF -> 220nF; LCSC C14663 -> C107083; MPN CC0603KRX7R9BB104 -> CC0603KRX7R9BB224; Note VIN high-frequency bypass, next to the VIN and PGND pins -> VIN high-frequency bypass, 50 V X7R, next to the VIN and PG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
- J7: footprint Combined_Local:CONN-TH_P3.96_HT396R-3.96-2P -> Combined_Local:CONN-TH_P3.96_HT396V-3.96-2P; LCSC C577799 -> C577788; MPN HT396R-3.96-2P -> HT396V-3.96-2P; Note 1 GND, 2 +24V, from the Wago split of the 24 V supply -> Kefa HT396V vertical header; mating plug HT396K-3.96-2P (C5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
- U6: value ADS1115IDGSR -> ADS1115IDGST; LCSC C37593 -> C468683; MPN ADS1115IDGSR -> ADS1115IDGST
Other:
- note added: "H1 to H5: M2.5 mounting holes, 2.7mm NPTH, not connected. H2 sits on the mains side: nylon screw and standoff, at least 5 mm tall."
- note removed: "H1, H2, H3: M2.5 mounting holes, 2.7mm NPTH, not connected. H2 sits on the mains side: nylon screw and standoff, at least 5 mm tall."

Commit message: Add H6 on the combined mains side and drop the nylon hardware
H6, a sixth M2.5 mounting hole, sits low in the 230 VAC area. From the
edge of the hardware (2.9 mm radius, a 5 mm hex standoff), H2 is 8.8 mm
from the mains copper and H6 9.6 mm from it and 12.5 mm from the GND
plane: each gap clears the 7 mm reinforced distance alone, so both take
metal screws and standoffs into the floating brass inserts. H1, H4 and
H5 have only GND plane under their hardware and need no keepout.

Co-Authored-By: Claude Opus 5.5 <noreply@anthropic.com>
Parts:
- added H6: M2.5, MountingHole:MountingHole_2.7mm_M2.5, symbol Mechanical:MountingHole
Other:
- note added: "H1 to H6: M2.5 mounting holes, 2.7mm NPTH, not connected. Metal screws and standoffs: the hardware edge of H2 and H6 stays more than 7 mm from mains and low-voltage copper."
- note removed: "H1 to H5: M2.5 mounting holes, 2.7mm NPTH, not connected. H2 sits on the mains side: nylon screw and standoff, at least 5 mm tall."
Changed lines of the file:
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@@
 		)
 	)
-	(text "H1 to H5: M2.5 mounting holes, 2.7mm NPTH, not connected.\nH2 sits on the mains side: nylon screw and standoff,\nat least 5 mm tall."
+	(text "H1 to H6: M2.5 mounting holes, 2.7mm NPTH, not connected.\nMetal screws and standoffs: the hardware edge of H2 and H6\nstays more than 7 mm from mains and low-voltage copper."
 		(exclude_from_sim no)
-		(at 320 245 0)
+		(at 320 255 0)
 		(effects
 			(font
@@
 					(unit 1)
 				)
+			)
+		)
+	)
+	(symbol
+		(lib_id "Mechanical:MountingHole")
+		(at 322.58 243.84 0)
+		(unit 1)
+		(body_style 1)
+		(exclude_from_sim no)
+		(in_bom no)
+		(on_board yes)
+		(in_pos_files yes)
+		(dnp no)
+		(property "Reference" "H6"
+			(at 327.58 241.84 0)
+			(show_name no)
+			(do_not_autoplace no)
+			(effects
+				(font
+					(size 1.1 1.1)
+				)
+				(justify left)
+			)
+		)
+		(property "Value" "M2.5"
+			(at 327.58 244.84 0)
+			(show_name no)
+			(do_not_autoplace no)
+			(effects
+				(font
+					(size 1 1)
+				)
+				(justify left)
+			)
+		)
+		(property "Footprint" "MountingHole:MountingHole_2.7mm_M2.5"
+			(at 322.58 243.84 0)
+			(hide yes)
+			(show_name no)
+			(do_not_autoplace no)
+			(effects
+				(font
+					(size 1 1)
+				)
+				(justify left)
+			)
+		)
+		(property "Datasheet" ""
+			(at 322.58 243.84 0)
+			(hide yes)
+			(show_name no)
+			(do_not_autoplace no)
+			(effects
+				(font
+					(size 1 1)
+				)
+				(justify left)
+			)
+		)
+		(property "Description" "Mounting Hole without connection"
+			(at 322.58 243.84 0)
+			(hide yes)
+			(show_name no)
+			(do_not_autoplace no)
+			(effects
+				(font
+					(size 1 1)
+				)
+				(justify left)
+			)
+		)
+		(property "MPN" "M2.5 / 2.7mm"
+			(at 322.58 243.84 0)
+			(hide yes)
+			(show_name no)
+			(do_not_autoplace no)
+			(effects
+				(font
+					(size 1 1)
+				)
+				(justify left)
+			)
+		)
+		(instances
+			(project "combined"
+				(path "/a3ee807d-f8aa-4db3-ad94-73a886b6ed37/a559a4b4-f0a6-43cb-a3de-d40c2438cf59"
+					(reference "H6")
+					(unit 1)
+				)

Commit message: Move combined to basic passives, M2 holes and an HT3.96 flow connector
- Mounting holes H1 to H6 become M2 (2.2 mm NPTH) and move on the board;
  the AC wing narrows to 35 mm.
- Nine extended passives become JLCPCB basic parts: R3 150, R5/R6
  300 + 300, R7 100 (1206 kept: an 0805 breaks the 1.5 mm L-side
  clearance), FB divider 120k/30k (5.00 V), EN divider 330k/24k
  (18.2 V / 16.7 V), C1 10 uF 1206, C5 220 nF 0805, setpoint filter
  1.5k / 2.2 uF. Only C2 (10 nF 1 kV) stays extended.
- J6 (flow) becomes a Kefa HT396V-3.96-3P: the Digmesa 0.5 mm2 wires
  screw into the plug without the JST-SM to XH adapter. Footprint and
  3D model from LCSC, checked against the Kefa drawing.
- The MPB003 manufacturer datasheet replaces gearpump.pdf; it confirms
  the 7-wire pinout used on J9.

Co-Authored-By: Claude Opus 5.5 <noreply@anthropic.com>
Parts:
- C1: footprint Capacitor_SMD:C_1210_3225Metric -> Capacitor_SMD:C_1206_3216Metric; LCSC C138687 -> C13585; MPN CL32B106KBJNNNE -> CL31A106KBHNNNE; Note VIN ceramic, X7R 50 V 1210 -> VIN ceramic, X5R 50 V 1206
- C5: footprint Capacitor_SMD:C_0603_1608Metric -> Capacitor_SMD:C_0805_2012Metric; LCSC C107083 -> C5378; MPN CC0603KRX7R9BB224 -> CL21B224KBFNNNE; Note VIN high-frequency bypass, 50 V X7R, next to the VIN and PG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 -> VIN high-frequency bypass, 50 V X7R 0805, next to the VIN a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
- H1, H2, H3, H4, H5, H6: value M2.5 -> M2; footprint MountingHole:MountingHole_2.7mm_M2.5 -> MountingHole:MountingHole_2.2mm_M2; MPN M2.5 / 2.7mm -> M2 / 2.2mm
- R28: value 100k -> 120k; LCSC C25803 -> C25808; MPN 0603WAF1003T5E -> 0603WAF1203T5E; Note FB divider top: 1.0 V x (1 + 100/24.9) = 5.02 V -> FB divider top: 1.0 V x (1 + 120/30) = 5.00 V
- R29: value 24.9k -> 30k; LCSC C25962 -> C22984; MPN 0603WAF2492T5E -> 0603WAF3002T5E
- R30: value 100k -> 330k; LCSC C25803 -> C23137; MPN 0603WAF1003T5E -> 0603WAF3303T5E; Note EN divider top: starts at 18.4 V, stops at 16.9 V -> EN divider top: starts at 18.2 V, stops at 16.7 V
- R31: value 7.15k -> 24k; LCSC C25980 -> C23352; MPN 0603WAF7151T5E -> 0603WAF2402T5E
Other:
- note added: "H1 to H6: M2 mounting holes, 2.2mm NPTH, not connected. Metal screws and standoffs: the hardware edge of H2 and H6 stays more than 7 mm from mains and low-voltage copper."
- note added: "U10 LMR33630A, 400 kHz: 5.00 V with R28/R29 (120k / 30k). EN divider R30/R31 (330k / 24k): starts at 18.2 V, stops at 16.7 V. +5V feeds J1 (screen), CAN, FLOW and the boiler SSR output. The XIAO 5V pin is VBUS of its USB-C, with no diode: never plug USB into the XIAO on this board. USB would drive +5V and, through the buck high-side body diode, the 24 V rail. Flash it off the board. XIAO 3V3 supp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"
- note removed: "H1 to H6: M2.5 mounting holes, 2.7mm NPTH, not connected. Metal screws and standoffs: the hardware edge of H2 and H6 stays more than 7 mm from mains and low-voltage copper."
- note removed: "U10 LMR33630A, 400 kHz: 5.02 V with R28/R29 (100k / 24.9k). EN divider R30/R31 (100k / 7.15k): starts at 18.4 V, stops at 16.9 V. +5V feeds J1 (screen), CAN, FLOW and the boiler SSR output. The XIAO 5V pin is VBUS of its USB-C, with no diode: never plug USB into the XIAO on this board. USB would drive +5V and, through the buck high-side body diode, the 24 V rail. Flash it off the board. XIAO 3V3 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"
Changed lines of the file:
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@@
 		)
 	)
-	(text "U10 LMR33630A, 400 kHz: 5.02 V with R28/R29 (100k / 24.9k). EN divider R30/R31 (100k / 7.15k):\nstarts at 18.4 V, stops at 16.9 V. +5V feeds J1 (screen), CAN, FLOW and the boiler SSR output.\nThe XIAO 5V pin is VBUS of its USB-C, with no diode: never plug USB into the XIAO on this board.\nUSB would drive +5V and, through the buck high-side body diode, the 24 V rail. Flash it off the board.\nXIAO 3V3 supplies CAN VIO, I2C, TMP102, ADS1115, FLOW pull-up, the valve driver\nand the PUMP_TACHO pull-up. USB-C, LDO, BOOT and RESET are on the removable XIAO."
+	(text "U10 LMR33630A, 400 kHz: 5.00 V with R28/R29 (120k / 30k). EN divider R30/R31 (330k / 24k):\nstarts at 18.2 V, stops at 16.7 V. +5V feeds J1 (screen), CAN, FLOW and the boiler SSR output.\nThe XIAO 5V pin is VBUS of its USB-C, with no diode: never plug USB into the XIAO on this board.\nUSB would drive +5V and, through the buck high-side body diode, the 24 V rail. Flash it off the board.\nXIAO 3V3 supplies CAN VIO, I2C, TMP102, ADS1115, FLOW pull-up, the valve driver\nand the PUMP_TACHO pull-up. USB-C, LDO, BOOT and RESET are on the removable XIAO."
 		(exclude_from_sim no)
 		(at 18 90 0)
@@
 		)
 	)
-	(text "H1 to H6: M2.5 mounting holes, 2.7mm NPTH, not connected.\nMetal screws and standoffs: the hardware edge of H2 and H6\nstays more than 7 mm from mains and low-voltage copper."
+	(text "H1 to H6: M2 mounting holes, 2.2mm NPTH, not connected.\nMetal screws and standoffs: the hardware edge of H2 and H6\nstays more than 7 mm from mains and low-voltage copper."
 		(exclude_from_sim no)
 		(at 320 255 0)
@@
 			)
 		)
-		(property "Value" "M2.5"
+		(property "Value" "M2"
 			(at 327.58 234.68 0)
 			(show_name no)
@@
 			)
 		)
-		(property "Footprint" "MountingHole:MountingHole_2.7mm_M2.5"
+		(property "Footprint" "MountingHole:MountingHole_2.2mm_M2"
 			(at 322.58 233.68 0)
 			(hide yes)
@@
 			)
 		)
-		(property "MPN" "M2.5 / 2.7mm"
+		(property "MPN" "M2 / 2.2mm"
 			(at 322.58 233.68 0)
 			(hide yes)
@@
 			)
 		)
-		(property "Value" "M2.5"
+		(property "Value" "M2"
 			(at 327.58 244.84 0)
 			(show_name no)
@@
 			)
 		)
-		(property "Footprint" "MountingHole:MountingHole_2.7mm_M2.5"
+		(property "Footprint" "MountingHole:MountingHole_2.2mm_M2"
 			(at 322.58 243.84 0)
 			(hide yes)
@@
 			)
 		)
-		(property "MPN" "M2.5 / 2.7mm"
+		(property "MPN" "M2 / 2.2mm"
 			(at 322.58 243.84 0)
 			(hide yes)
@@
 			)
 		)
-		(property "Value" "M2.5"
+		(property "Value" "M2"
 			(at 327.58 224.52 0)
 			(show_name no)
@@
 			)
 		)
-		(property "Footprint" "MountingHole:MountingHole_2.7mm_M2.5"
+		(property "Footprint" "MountingHole:MountingHole_2.2mm_M2"
 			(at 322.58 223.52 0)
 			(hide yes)
@@
 			)
 		)
-		(property "MPN" "M2.5 / 2.7mm"
+		(property "MPN" "M2 / 2.2mm"
 			(at 322.58 223.52 0)
 			(hide yes)
@@
 			)
 		)
-		(property "Value" "M2.5"
+		(property "Value" "M2"
 			(at 327.58 214.36 0)
 			(show_name no)
@@
 			)
 		)
-		(property "Footprint" "MountingHole:MountingHole_2.7mm_M2.5"
+		(property "Footprint" "MountingHole:MountingHole_2.2mm_M2"
 			(at 322.58 213.36 0)
 			(hide yes)
@@
 			)
 		)
-		(property "MPN" "M2.5 / 2.7mm"
+		(property "MPN" "M2 / 2.2mm"
 			(at 322.58 213.36 0)
 			(hide yes)
@@
 			)
 		)
-		(property "Value" "M2.5"
+		(property "Value" "M2"
 			(at 327.58 204.2 0)
 			(show_name no)
@@
 			)
 		)
-		(property "Footprint" "MountingHole:MountingHole_2.7mm_M2.5"
+		(property "Footprint" "MountingHole:MountingHole_2.2mm_M2"
 			(at 322.58 203.2 0)
 			(hide yes)
@@
 			)
 		)
-		(property "MPN" "M2.5 / 2.7mm"
+		(property "MPN" "M2 / 2.2mm"
 			(at 322.58 203.2 0)
 			(hide yes)
@@
 			)
 		)
-		(property "Value" "M2.5"
+		(property "Value" "M2"
 			(at 327.58 194.04 0)
 			(show_name no)
@@
 			)
 		)
-		(property "Footprint" "MountingHole:MountingHole_2.7mm_M2.5"
+		(property "Footprint" "MountingHole:MountingHole_2.2mm_M2"
 			(at 322.58 193.04 0)
 			(hide yes)
@@
 			)
 		)
-		(property "MPN" "M2.5 / 2.7mm"
+		(property "MPN" "M2 / 2.2mm"
 			(at 322.58 193.04 0)
 			(hide yes)
@@
 			)
 		)
-		(property "Footprint" "Capacitor_SMD:C_1210_3225Metric"
+		(property "Footprint" "Capacitor_SMD:C_1206_3216Metric"
 			(at 53.34 46.99 0)
 			(hide yes)
@@
 			)
 		)
-		(property "MPN" "CL32B106KBJNNNE"
+		(property "MPN" "CL31A106KBHNNNE"
 			(at 53.34 46.99 0)
 			(hide yes)
@@
 			)
 		)
-		(property "LCSC" "C138687"
+		(property "LCSC" "C13585"
 			(at 53.34 46.99 0)
 			(hide yes)
@@
 			)
 		)
-		(property "Note" "VIN ceramic, X7R 50 V 1210"
+		(property "Note" "VIN ceramic, X5R 50 V 1206"
 			(at 53.34 46.99 0)
 			(hide yes)
@@
 			)
 		)
-		(property "Footprint" "Capacitor_SMD:C_0603_1608Metric"
+		(property "Footprint" "Capacitor_SMD:C_0805_2012Metric"
 			(at 83.82 46.99 0)
 			(hide yes)
@@
 			)
 		)
-		(property "MPN" "CC0603KRX7R9BB224"
+		(property "MPN" "CL21B224KBFNNNE"
 			(at 83.82 46.99 0)
 			(hide yes)
@@
 			)
 		)
-		(property "LCSC" "C107083"
+		(property "LCSC" "C5378"
 			(at 83.82 46.99 0)
 			(hide yes)
@@
 			)
 		)
-		(property "Note" "VIN high-frequency bypass, 50 V X7R, next to the VIN and PGND pins"
+		(property "Note" "VIN high-frequency bypass, 50 V X7R 0805, next to the VIN and PGND pins"
 			(at 83.82 46.99 0)
 			(hide yes)
@@
 			)
 		)
-		(property "Value" "100k"
+		(property "Value" "330k"
 			(at 116.84 45.72 0)
 			(show_name no)
@@
 			)
 		)
-		(property "MPN" "0603WAF1003T5E"
+		(property "MPN" "0603WAF3303T5E"
 			(at 114.3 44.45 0)
 			(hide yes)
@@
 			)
 		)
-		(property "LCSC" "C25803"
+		(property "LCSC" "C23137"
 			(at 114.3 44.45 0)
 			(hide yes)
@@
 			)
 		)
-		(property "Note" "EN divider top: starts at 18.4 V, stops at 16.9 V"
+		(property "Note" "EN divider top: starts at 18.2 V, stops at 16.7 V"
 			(at 114.3 44.45 0)
 			(hide yes)
@@
 			)
 		)
-		(property "Value" "7.15k"
+		(property "Value" "24k"
 			(at 111.76 53.34 0)
 			(show_name no)
@@
 			)
 		)
-		(property "MPN" "0603WAF7151T5E"
+		(property "MPN" "0603WAF2402T5E"
 			(at 114.3 52.07 0)
 			(hide yes)
@@
 			)
 		)
-		(property "LCSC" "C25980"
+		(property "LCSC" "C23352"
 			(at 114.3 52.07 0)
 			(hide yes)
@@
 			)
 		)
-		(property "Value" "100k"
+		(property "Value" "120k"
 			(at 181.61 48.26 0)
 			(show_name no)
@@
 			)
 		)
-		(property "MPN" "0603WAF1003T5E"
+		(property "MPN" "0603WAF1203T5E"
 			(at 179.07 46.99 0)
 			(hide yes)
@@
 			)
 		)
-		(property "LCSC" "C25803"
+		(property "LCSC" "C25808"
 			(at 179.07 46.99 0)
 			(hide yes)
@@
 			)
 		)
-		(property "Note" "FB divider top: 1.0 V x (1 + 100/24.9) = 5.02 V"
+		(property "Note" "FB divider top: 1.0 V x (1 + 120/30) = 5.00 V"
 			(at 179.07 46.99 0)
 			(hide yes)
@@
 			)
 		)
-		(property "Value" "24.9k"
+		(property "Value" "30k"
 			(at 181.61 55.88 0)
 			(show_name no)
@@
 			)
 		)
-		(property "MPN" "0603WAF2492T5E"
+		(property "MPN" "0603WAF3002T5E"
 			(at 179.07 54.61 0)
 			(hide yes)
@@
 			)
 		)
-		(property "LCSC" "C25962"
+		(property "LCSC" "C22984"
 			(at 179.07 54.61 0)
 			(hide yes)
